File: PCB/PoolMonitor.kicad_sch (KiCad schematic)
At the start: 28 parts, among them J1 Conn_01x02_Male, J2 Conn_01x06_Female, J3 SolarPanel6V, Q1 DMP2225L-7, Q2 AO3400A, U1 K7803M-1000R3, U2 ESP-12E

Commit message: Updated to use all JST connectors and updated REAME with a description
Parts:
- TempSense1: footprint Connector_Molex:Molex_SPOX_5267-03A_1x03_P2.50mm_Vertical -> Connector_JST:JST_PH_B3B-PH-K_1x03_P2.00mm_Vertical; LCSC C293315 -> C131339
Changed lines of the file:
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@@
       (effects (font (size 1.27 1.27)) (justify right))
     )
-    (property "Footprint" "Connector_Molex:Molex_SPOX_5267-03A_1x03_P2.50mm_Vertical" (id 2) (at 132.08 22.86 0)
+    (property "Footprint" "Connector_JST:JST_PH_B3B-PH-K_1x03_P2.00mm_Vertical" (id 2) (at 132.08 22.86 0)
       (effects (font (size 1.27 1.27)) hide)
     )
@@
       (effects (font (size 1.27 1.27)) hide)
     )
-    (property "LCSC" "C293315" (id 4) (at 132.08 22.86 0)
+    (property "LCSC" "C131339" (id 4) (at 132.08 22.86 0)
       (effects (font (size 1.27 1.27)) hide)
     )
@@
     )
     (path "/00000000-0000-0000-0000-000060c07b2c"
-      (reference "TempSense1") (unit 1) (value "Conn_01x03_Male") (footprint "Connector_Molex:Molex_SPOX_5267-03A_1x03_P2.50mm_Vertical")
+      (reference "TempSense1") (unit 1) (value "Conn_01x03_Male") (footprint "Connector_JST:JST_PH_B3B-PH-K_1x03_P2.00mm_Vertical")
     )
     (path "/7d02c8da-c1f5-46b6-a684-03b1f9fa82ce"
